File: Eagle/charger board v3/preroute/charger_v3.sch (EAGLE design)
At the start: 37 parts, among them IC1 IR2110D, Q2 IRFP240, Q3 MJE13003G

Commit message: routing v3
routing v3: opto, snubber, momentary pb, fuse adjst
Parts:
- removed C5, C6: 22uF, rcl:CPOL-EUE7.5-18
- removed LM35: JST-XH-03-PIN-LONG-PAD, Rembrandt Electronics - JST XH Connectors v1-0:JST-XH-03-PIN-LONG-PAD
- removed OK1: SFH618A-5, optocoupler:SFH618A-5
- removed R7: 1k, rcl:R-US_0204/7
- removed R8, R9: 31, rcl:R-US_0411/15
- removed S1: (no value), switch-omron:10-XX
- added IC2: LM35CZ, lm35:LM35CZ
- added Q1: 2N7000, 2N7000:2N7000
- added U$1: SWITCH-DPDT-7X7A, TA_library:SWITCH-DPDT-7X7A
- AC_IN: value 1977477-2 -> XT90A; device terminal_block_TA:1977477-2 -> TA_library:XT90A
- F1: device TA_library:FUSEHOLDER -> fuse:SH25
- R1: value 180 -> 10k
- R4: device rcl:R-US_0411/15 -> rcl:R-US_0309/12
Connections:
- removed net N$11: OK1.COL, R1.2
- removed net N$6: C5.+, R8.1
- removed net N$7: C6.-, R9.2
- net 5V: now also IC2.+VS, R1.2; no longer LM35-3.S, R1.1
- net AC_1: now also AC_IN.IN_1; no longer AC_IN.1
- net AC_2: now also AC_IN.IN_2; no longer AC_IN.2
- net GND: now also DC_OUT.2, IC2.GND, Q1.S; no longer C6.+, DC_OUT.1, LM35-1.S, OK1.C, R7.1
- net HVDC: now also U$1.1; no longer R8.2, S1.S1
- net N$2: now also U$1.2; no longer S1.P
- net NMOS_SOURCE: no longer C5.-, R9.1
- net PWM_5V: now also Q1.D, R1.1; no longer OK1.EMIT, R7.2
- net PWM_SW1: now also Q1.G; no longer OK1.A
- net TEMP: now also IC2.VO; no longer LM35-2.S
- net V_OUT_FUSE: now also DC_OUT.1; no longer DC_OUT.2
Other:
- moved on the sheet: AC_IN, C3, R1
