File: Eagle/charger board v4/charger_v4.brd (EAGLE design)
At the start: 195.2 x 133.3 mm, 61 parts, among them IC1 IR2110D, Q2 IRFP240, Q3 MJE13003G

Commit message: Update routing charger v4
Parts:
- added TEMP: JST-XH-03-PIN-LONG-PAD, JST XH Connectors v1-0:JST-XH-03-PACKAGE-LONG-PAD
- moved GND1 7.62 mm to (8.89, 90.2)
- moved P_5V 7.62 mm to (26.7, 90.2)
- moved GND2 7.62 mm to (8.89, 102.9)
- moved P_3V3 7.62 mm to (26.7, 102.9)
- moved R14 2.54 mm to (50.8, 125.7)
- moved R15 2.54 mm to (35.6, 125.7)
- moved D2 2.54 mm to (80.0, 82.5)
- moved R2 2.54 mm to (74.9, 82.5)
- moved R3 2.54 mm to (69.8, 82.5)
- moved L2 1.65 mm to (99.1, 93.1)
- moved L1 1.42 mm to (128.1, 40.4)
- moved D4 1.27 mm to (24.1, 78.7)
- moved P_IR 1.27 mm to (82.5, 91.4)
- moved R6 1.27 mm to (33.0, 78.7)
- moved S1 1.27 mm to (14.0, 78.7)
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- renumbered U$1 to DRAIN_JUMP, U$2 to SOURCE_JUMP, U$3 to NMOS_SNUB_JUMP, U$4 to DIODE_SNUB_JUMP, U$5 to DC_OUTPUT, U$6 to INDUCTOR_JUMP, U$7 to AC_INPUT, U$8 to ACS_INPUTS
Connections:
- net 5V: now also TEMP.1
- net GND: now also TEMP.3
- net TEMP_SENSE: now also TEMP.2
Routing:
- net GND: track 385.5 -> 701.6 mm
- net 5V: track 0.00 -> 207.1 mm, vias 0 -> 1
- net PWM_DISCHARGE: track 0.00 -> 123.6 mm
- net CURRENT_SENSE: track 0.00 -> 108.1 mm
- net TEMP_SENSE: track 0.00 -> 73.9 mm, vias 0 -> 1
- net PWM_MOSFET: track 0.00 -> 56.9 mm
- net PWM_OPTO: track 0.00 -> 47.6 mm
- net VOLTAGE_SENSE: track 0.00 -> 45.2 mm
- net NMOS_SOURCE: track 193.5 -> 238.7 mm
- net HV_SENSE: track 0.00 -> 40.8 mm
- net HVDC: track 84.4 -> 117.0 mm
- net 12V: track 12.8 -> 32.6 mm
- net NMOS_DRAIN: track 104.0 -> 121.5 mm
- net PWM_IR: track 35.9 -> 53.3 mm
- net N$9: track 0.00 -> 12.0 mm
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- added copper zone on layer 1, net GND
- added copper zone on layer 16, net GND
Other:
- board text added: "AC Cap Discharge"
- board text added: "CHARGER V4 Dhanu Danu Naoko"
- board text added: "Eren"
- board text added: "IP+"
- board text added: "IP-"
- board text removed: "Charger V4"
