File: Eagle/charger board v4/charger_v4.sch (EAGLE design)
At the start: 61 parts, among them IC1 IR2110D, Q2 IRFP240, Q3 MJE13003G

Commit message: Update routing charger v4
Parts:
- added TEMP: JST-XH-03-PIN-LONG-PAD, JST XH Connectors v1-0:JST-XH-03-PIN-LONG-PAD
- renumbered U$1 to DRAIN_JUMP, U$2 to SOURCE_JUMP, U$3 to NMOS_SNUB_JUMP, U$4 to DIODE_SNUB_JUMP, U$5 to DC_OUTPUT, U$6 to INDUCTOR_JUMP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
Connections:
- net 5V: now also TEMP-1.S
- net GND: now also TEMP-3.S
- net TEMP_SENSE: now also TEMP-2.S
