File: Eagle/Kontrol v2/kontrol_v2.brd (EAGLE design)
At the start: 83.2 x 77.4 mm, 21 parts, among them J1 1977477-2, X1 JST-XH-06-PIN-LONG-PAD, X10 JST-XH-02-PIN-LONG-PAD, X11 JST-XH-02-PIN-LONG-PAD, X12 JST-XH-02-PIN-LONG-PAD, X2 JST-XH-06-PIN-LONG-PAD, X3 JST-XH-04-PIN-LONG-PAD, X4 JST-XH-04-PIN-LONG-PAD, X5 JST-XH-04-PIN-LONG-PAD, X6 JST-XH-04-PIN-LONG-PAD, X8 JST-XH-03-PIN-LONG-PAD, X9 JST-XH-02-PIN-LONG-PAD

Commit message: edit kontrol v2
Parts:
- removed X2: JST-XH-06-PIN-LONG-PAD, JST XH Connectors v1-0:JST-XH-06-PACKAGE-LONG-PAD
- removed X4: JST-XH-04-PIN-LONG-PAD, JST XH Connectors v1-0:JST-XH-04-PACKAGE-LONG-PAD
Connections:
- removed net RX_TESTERBOARD: U$1.16
- removed net TEMP: X2.5
- removed net TX_TESTERBOARD: U$1.17
- new net 5V_ESP: U$1.19
- new net CUR_SENSE: X3.3
- new net PWM_DISCHARGE: X1.4
- new net PWM_MOSFET: X1.3
- new net VOL_SENSE: X3.4
- net 12V: no longer X2.1
- net 5V: no longer U$1.19, X2.2, X4.1
- net CUR_SENSE_1: no longer X3.3
- net CUR_SENSE_2: no longer X4.3
- net GND: no longer X2.6, X4.2
- net PWM_DISCHARGE_KANAN: no longer X2.4
- net PWM_DISCHARGE_KIRI: no longer X1.4
- net PWM_MOSFET_KANAN: no longer X2.3
- net PWM_MOSFET_KIRI: no longer X1.3
- net VOL_SENSE_1: no longer X3.4
- net VOL_SENSE_2: no longer X4.4
Changed lines of the file:
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@@
 </element>
 <element name="X1" library="JST XH Connectors v1-0" package="JST-XH-06-PACKAGE-LONG-PAD" value="JST-XH-06-PIN-LONG-PAD" x="39.1414" y="23.6982" smashed="yes"/>
-<element name="X2" library="JST XH Connectors v1-0" package="JST-XH-06-PACKAGE-LONG-PAD" value="JST-XH-06-PIN-LONG-PAD" x="57.6326" y="23.6728" smashed="yes"/>
 <element name="X3" library="JST XH Connectors v1-0" package="JST-XH-04-PACKAGE-LONG-PAD" value="JST-XH-04-PIN-LONG-PAD" x="83.9978" y="59.2074" smashed="yes" rot="R90"/>
-<element name="X4" library="JST XH Connectors v1-0" package="JST-XH-04-PACKAGE-LONG-PAD" value="JST-XH-04-PIN-LONG-PAD" x="84.0232" y="73.8378" smashed="yes" rot="R90"/>
 <element name="JP4" library="pinhead" library_urn="urn:adsk.eagle:library:325" package="1X10" package3d_urn="urn:adsk.eagle:package:22406/2" value="" x="76.6318" y="84.5312" smashed="yes" rot="R270">
 <attribute name="POPULARITY" value="35" x="76.6318" y="84.5312" size="1.778" layer="27" rot="R270" display="off"/>
@@
 <contactref element="MINI1" pad="IN-2"/>
 <contactref element="MINI1" pad="IN-3"/>
-<contactref element="X2" pad="6"/>
 <contactref element="X3" pad="2"/>
-<contactref element="X4" pad="2"/>
 <contactref element="JP4" pad="2"/>
 <contactref element="JP4" pad="5"/>
@@
 <wire x1="76.6318" y1="85.8012" x2="76.6318" y2="93.4212" width="0" layer="19" extent="1-1"/>
 <wire x1="84.0486" y1="85.8774" x2="76.6318" y2="85.8012" width="0" layer="19" extent="1-1"/>
-<wire x1="84.0232" y1="72.5678" x2="84.0486" y2="85.8774" width="0" layer="19" extent="1-1"/>
-<wire x1="76.7334" y1="62.103" x2="84.0232" y2="72.5678" width="0" layer="19" extent="1-1"/>
+<wire x1="76.7334" y1="62.103" x2="76.6318" y2="85.8012" width="0" layer="19" extent="1-1"/>
 <wire x1="83.9978" y1="57.9374" x2="76.7334" y2="62.103" width="0" layer="19" extent="1-1"/>
 <wire x1="59.93" y1="60.72" x2="76.7334" y2="62.103" width="0" layer="19" extent="1-1"/>
@@
 <wire x1="57.39" y1="30.24" x2="57.39" y2="32.78" width="0" layer="19" extent="1-1"/>
 <wire x1="45.4914" y1="23.6982" x2="57.39" y2="30.24" width="0" layer="19" extent="1-1"/>
-<wire x1="63.9826" y1="23.6728" x2="59.93" y2="30.24" width="0" layer="19" extent="1-1"/>
-<wire x1="36.8908" y1="35.9378" x2="52.1308" y2="35.9378" width="0" layer="19" extent="1-1"/>
-<wire x1="37.2618" y1="31.4546" x2="36.8908" y2="35.9378" width="0" layer="19" extent="1-1"/>
+<wire x1="37.2618" y1="31.4546" x2="45.4914" y2="23.6982" width="0" layer="19" extent="1-1"/>
+<wire x1="36.8908" y1="35.9378" x2="37.2618" y2="31.4546" width="0" layer="19" extent="1-1"/>
 <wire x1="19.3802" y1="23.6728" x2="37.2618" y2="31.4546" width="0" layer="19" extent="1-1"/>
 <wire x1="5.842" y1="23.6474" x2="19.3802" y2="23.6728" width="0" layer="19" extent="1-1"/>
@@
 </signal>
 <signal name="5V">
-<contactref element="U$1" pad="19"/>
 <contactref element="C2" pad="1"/>
 <contactref element="C1" pad="1"/>
 <contactref element="X1" pad="2"/>
-<contactref element="X2" pad="2"/>
 <contactref element="X3" pad="1"/>
-<contactref element="X4" pad="1"/>
 <contactref element="JP4" pad="1"/>
 <contactref element="JP5" pad="1"/>
@@
 <contactref element="MINI1" pad="OUT+3"/>
 <contactref element="JP1" pad="7"/>
-<wire x1="76.6318" y1="95.9612" x2="84.0232" y2="70.0278" width="0" layer="19" extent="1-1"/>
-<wire x1="83.9978" y1="55.3974" x2="76.6318" y2="95.9612" width="0" layer="19" extent="1-1"/>
-<wire x1="76.7334" y1="54.483" x2="83.9978" y2="55.3974" width="0" layer="19" extent="1-1"/>
-<wire x1="76.7334" y1="64.643" x2="76.7334" y2="54.483" width="0" layer="19" extent="1-1"/>
-<wire x1="34.7218" y1="31.4546" x2="76.7334" y2="64.643" width="0" layer="19" extent="1-1"/>
-<wire x1="72.63" y1="32.78" x2="34.7218" y2="31.4546" width="0" layer="19" extent="1-1"/>
+<wire x1="76.7334" y1="64.643" x2="76.6318" y2="95.9612" width="0" layer="19" extent="1-1"/>
+<wire x1="76.7334" y1="54.483" x2="76.7334" y2="64.643" width="0" layer="19" extent="1-1"/>
+<wire x1="83.9978" y1="55.3974" x2="76.7334" y2="54.483" width="0" layer="19" extent="1-1"/>
+<wire x1="72.63" y1="32.78" x2="76.7334" y2="54.483" width="0" layer="19" extent="1-1"/>
 <wire x1="70.09" y1="32.78" x2="72.63" y2="32.78" width="0" layer="19" extent="1-1"/>
 <wire x1="72.63" y1="30.24" x2="72.63" y2="32.78" width="0" layer="19" extent="1-1"/>
 <wire x1="70.09" y1="30.24" x2="70.09" y2="32.78" width="0" layer="19" extent="1-1"/>
-<wire x1="53.8226" y1="23.6728" x2="70.09" y2="30.24" width="0" layer="19" extent="1-1"/>
-<wire x1="35.3314" y1="23.6982" x2="53.8226" y2="23.6728" width="0" layer="19" extent="1-1"/>
-<wire x1="12.4778" y1="63.6504" x2="35.3314" y2="23.6982" width="0" layer="19" extent="1-1"/>
+<wire x1="35.3314" y1="23.6982" x2="70.09" y2="30.24" width="0" layer="19" extent="1-1"/>
+<wire x1="34.7218" y1="31.4546" x2="35.3314" y2="23.6982" width="0" layer="19" extent="1-1"/>
+<wire x1="12.4778" y1="63.6504" x2="34.7218" y2="31.4546" width="0" layer="19" extent="1-1"/>
 <wire x1="7.0604" y1="63.6758" x2="12.4778" y2="63.6504" width="0" layer="19" extent="1-1"/>
-<wire x1="6.4108" y1="58.5878" x2="7.0604" y2="63.6758" width="0" layer="19" extent="1-1"/>
 </signal>
 <signal name="TX">
@@
 <contactref element="MINI1" pad="IN+3"/>
 <contactref element="X1" pad="1"/>
-<contactref element="X2" pad="1"/>
 <contactref element="X8" pad="3"/>
 <wire x1="70.51" y1="66.5" x2="84.0486" y2="88.4174" width="0" layer="19" extent="1-1"/>
@@
 <wire x1="72.63" y1="58.18" x2="72.63" y2="60.72" width="0" layer="19" extent="1-1"/>
 <wire x1="70.09" y1="58.18" x2="70.09" y2="60.72" width="0" layer="19" extent="1-1"/>
-<wire x1="51.2826" y1="23.6728" x2="70.09" y2="58.18" width="0" layer="19" extent="1-1"/>
-<wire x1="32.7914" y1="23.6982" x2="51.2826" y2="23.6728" width="0" layer="19" extent="1-1"/>
+<wire x1="32.7914" y1="23.6982" x2="70.09" y2="58.18" width="0" layer="19" extent="1-1"/>
 </signal>
 <signal name="PWM_MOSFET_KIRI">
-<contactref element="X1" pad="3"/>
 <contactref element="U$1" pad="28"/>
-<wire x1="26.7308" y1="35.9378" x2="37.8714" y2="23.6982" width="0" layer="19" extent="1-1"/>
 </signal>
 <signal name="PWM_DISCHARGE_KIRI">
-<contactref element="X1" pad="4"/>
 <contactref element="U$1" pad="30"/>
-<wire x1="40.4114" y1="23.6982" x2="31.8108" y2="35.9378" width="0" layer="19" extent="1-1"/>
 </signal>
 <signal name="TEMP1">
@@
 </signal>
 <signal name="PWM_MOSFET_KANAN">
-<contactref element="X2" pad="3"/>
 <contactref element="U$1" pad="31"/>
-<wire x1="34.3508" y1="35.9378" x2="56.3626" y2="23.6728" width="0" layer="19" extent="1-1"/>
 </signal>
 <signal name="PWM_DISCHARGE_KANAN">
-<contactref element="X2" pad="4"/>
 <contactref element="U$1" pad="37"/>
-<wire x1="49.5908" y1="35.9378" x2="58.9026" y2="23.6728" width="0" layer="19" extent="1-1"/>
-</signal>
-<signal name="TEMP">
-<contactref element="X2" pad="5"/>
 </signal>
 <signal name="CUR_SENSE_1">
-<contactref element="X3" pad="3"/>
 <contactref element="JP5" pad="7"/>
-<wire x1="76.7334" y1="49.403" x2="83.9978" y2="60.4774" width="0" layer="19" extent="1-1"/>
 </signal>
 <signal name="VOL_SENSE_1">
-<contactref element="X3" pad="4"/>
 <contactref element="JP5" pad="8"/>
-<wire x1="76.7334" y1="46.863" x2="83.9978" y2="63.0174" width="0" layer="19" extent="1-1"/>
 </signal>
 <signal name="CUR_SENSE_2">
-<contactref element="X4" pad="3"/>
 <contactref element="JP5" pad="9"/>
-<wire x1="76.7334" y1="44.323" x2="84.0232" y2="75.1078" width="0" layer="19" extent="1-1"/>
 </signal>
 <signal name="VOL_SENSE_2">
-<contactref element="X4" pad="4"/>
 <contactref element="JP5" pad="10"/>
-<wire x1="76.7334" y1="41.783" x2="84.0232" y2="77.6478" width="0" layer="19" extent="1-1"/>
 </signal>
 <signal name="SCL">
@@
 <contactref element="U$1" pad="15"/>
 </signal>
-<signal name="RX_TESTERBOARD">
-<contactref element="U$1" pad="16"/>
-</signal>
-<signal name="TX_TESTERBOARD">
-<contactref element="U$1" pad="17"/>
-</signal>
 <signal name="RED_KIRI">
 <contactref element="U$1" pad="23"/>
@@
 <contactref element="U$1" pad="7"/>
 </signal>
+<signal name="PWM_MOSFET">
+<contactref element="X1" pad="3"/>
+</signal>
+<signal name="PWM_DISCHARGE">
+<contactref element="X1" pad="4"/>
+</signal>
+<signal name="CUR_SENSE">
+<contactref element="X3" pad="3"/>
+</signal>
+<signal name="VOL_SENSE">
+<contactref element="X3" pad="4"/>
+</signal>
+<signal name="5V_ESP">
+<contactref element="U$1" pad="19"/>
+</signal>
 </signals>

Commit message: nambahin library eagle+update kontrolv2
Parts:
- removed J1: 1977477-2, terminal_block:TE_1977477-2
- removed JP1: (no value), pinhead:1X07
- removed JP5: (no value), pinhead:1X10
- removed X9: JST-XH-02-PIN-LONG-PAD, JST XH Connectors v1-0:JST-XH-02-PACKAGE-LONG-PAD
- added 1K: 1k, rcl:0204/7
- added 330: 6k, rcl:0204/7
- added C3: (no value), rcl:E2,5-6E
- added D4: (no value), Sparkfun_LED:LED_5MM
- added D7: UF4007, diode:DO34-7
- added JP3: (no value), pinhead:1X16
- added JP6: (no value), pinhead:1X09
- added JP7: (no value), pinhead:1X02
- added JP8: (no value), pinhead:1X01
- added K1: SRD-12VDC-SL-C, TA_library:RELAY_SRD-12VDC-SL-C
- added NPN: (no value), transistor:TO92-CBE
- added OVR_BMS: JST-XH-02-PIN-LONG-PAD, JST XH Connectors v1-0:JST-XH-02-PACKAGE-LONG-PAD
- added U$2: ADS1115, ADS1115:ADS1115
- added U$3: SIM800V2, sim800v2:SIM800V2
- added X2: JST-XH-03-PIN-LONG-PAD, JST XH Connectors v1-0:JST-XH-03-PACKAGE-LONG-PAD
- JP4: device pinhead:1X10 -> pinhead:1X01
- moved X10 116.7 mm to (16.5, 121.9)
- moved X11 107.8 mm to (25.4, 121.9), turned to 0 degrees
- moved X1 106.0 mm to (45.7, 129.5)
- moved X5 106.0 mm to (15.2, 129.5)
- moved X6 106.0 mm to (29.2, 129.5)
- moved JP2 79.5 mm to (63.3, 130.3)
- moved X12 77.7 mm to (59.7, 121.9), turned to 0 degrees
- moved X3 72.2 mm to (48.3, 121.9), turned to 0 degrees
- moved U$1 54.8 mm to (50.4, 97.7), turned to 0 degrees
- moved JP4 51.0 mm to (70.2, 33.9), turned to 0 degrees
- moved HI_LINK1 47.5 mm to (36.0, 20.2), turned to 180 degrees
- moved X8 38.7 mm to (69.8, 121.9), turned to 0 degrees
- moved C1 36.6 mm to (43.5, 68.3)
- moved C2 36.6 mm to (49.0, 68.3)
- moved MINI1 24.1 mm to (70.8, 41.7), turned to 90 degrees
Connections:
- removed net CUR_SENSE_1: JP5.7
- removed net CUR_SENSE_2: JP5.9
- removed net N$10: X10.2
- removed net N$12: X11.2
- removed net N$14: X12.2
- removed net N$2: HI_LINK1.AC-, J1.1
- removed net N$3: U$1.15
- removed net N$43: JP4.6
- removed net N$46: JP4.9
- removed net N$47: JP4.10
- removed net N$53: JP5.6
- removed net N$7: X9.2
- removed net PWM_DISCHARGE_KANAN: U$1.37
- removed net PWM_DISCHARGE_KIRI: U$1.30
- removed net PWM_MOSFET_KANAN: U$1.31
- removed net PWM_MOSFET_KIRI: U$1.28
- removed net TEMP2: JP4.8
- removed net VOL_SENSE_1: JP5.8
- removed net VOL_SENSE_2: JP5.10
- new net AC: K1.COM
- new net AC_IN_1: K1.NO
- new net EN: C3.+, U$1.2
- new net N$19: 1K.2, NPN.B
- new net N$21: D7.A, K1.COIL2, NPN.C
- new net N$23: JP3.14, U$1.25
- new net N$24: JP3.15, U$1.24
- new net N$44: JP8.1, U$2.A3
- new net N$9: JP6.3, U$1.13
- new net RELAY: 1K.1, D4.K, JP6.7, U$1.9
- new net RX_BMS: JP3.4, U$1.35
- new net RX_IOT: JP6.6, U$1.10
- new net TEMP: U$2.A2, X2.2
- new net TX_BMS: JP3.5, U$1.34
- new net TX_IOT: JP6.5, U$1.11
- net 12V: now also JP4.1
- net 5V: now also D7.C, JP7.1, K1.COIL1, U$2.5V, U$3.5V, X2.1; no longer JP1.7, JP4.1, JP5.1, JP5.5
- net 5V_ESP: now also JP7.2
- net BLU_KANAN: now also JP3.9, U$1.30; no longer U$1.29
- net BLU_KIRI: now also JP3.13, U$1.26; no longer U$1.25
- net CUR_SENSE: now also U$2.A0
- net DETEKSI_BATERAI_KANAN: now also JP6.8
- net DETEKSI_BATERAI_KIRI: now also JP6.9, U$1.7; no longer U$1.10
- net GND: now also 330.1, C3.-, JP3.1, JP3.7, NPN.E, OVR_BMS.2, U$2.ADDR, U$2.GND, U$3.GND, U$3.GND1, X10.2, X11.2, X12.2, X2.3; no longer JP1.6, JP4.2, JP4.5, JP5.2
- net GRN_KANAN: now also JP3.2, U$1.37; no longer U$1.27
- net GRN_KIRI: now also JP3.11, U$1.28; no longer U$1.24
- net N$1: now also 330.2, D4.A; no longer HI_LINK1.AC+, J1.2
- net N$8: now also JP6.2, U$1.14; no longer U$1.7
- net OVERRIDE_BMS: now also JP6.1, OVR_BMS.1, U$1.15; no longer U$1.11, X9.1
- net PWM_DISCHARGE: now also JP3.16, U$1.23
- net PWM_MOSFET: now also JP3.10, U$1.29
- net RED_KANAN: now also JP3.8, U$1.31; no longer U$1.26
- net RED_KIRI: now also JP3.12, U$1.27; no longer U$1.23
- net RX: now also U$3.RX; no longer JP1.4, U$1.34
- net SCL: now also JP3.3, U$2.SCL; no longer JP4.3, JP5.3
- net SDA: now also JP3.6, U$2.SDA; no longer JP4.4, JP5.4
- net SWITCH_MODE_DAYA: now also JP6.4, U$1.12; no longer U$1.9
- net TEMP1: no longer JP4.7
- net TX: now also U$3.TX; no longer JP1.3, U$1.35
- net VOL_SENSE: now also U$2.A1
Other:
- board size 83.2 x 77.4 mm -> 86.4 x 136.6 mm

Commit message: Update board kontrol
Harusnya sudah selesai
Parts:
- removed X1: JST-XH-06-PIN-LONG-PAD, JST XH Connectors v1-0:JST-XH-06-PACKAGE-LONG-PAD
- removed X10, X11, X12: JST-XH-02-PIN-LONG-PAD, JST XH Connectors v1-0:JST-XH-02-PACKAGE-LONG-PAD
- removed X2, X8: JST-XH-03-PIN-LONG-PAD, JST XH Connectors v1-0:JST-XH-03-PACKAGE-LONG-PAD
- removed X3, X5, X6: JST-XH-04-PIN-LONG-PAD, JST XH Connectors v1-0:JST-XH-04-PACKAGE-LONG-PAD
- added 5V: 5V, pinhead:1X05
- added C5: 2mF, rcl:E3,5-10
- added CHARGER: JST-XH-08-PIN-LONG-PAD, Rembrandt Electronics - JST XH Connectors v1-0:JST-XH-08-PACKAGE-LONG-PAD
- added CHGMODE, DB_L, DB_R: JST-XH-02-PIN-LONG-PAD, JST XH Connectors v1-0:JST-XH-02-PACKAGE-LONG-PAD
- added FAN, TEMP: JST-XH-03-PIN-LONG-PAD, JST XH Connectors v1-0:JST-XH-03-PACKAGE-LONG-PAD
- added GND: GND, pinhead:1X05
- added LED_L, LED_R, SENSING: JST-XH-04-PIN-LONG-PAD, JST XH Connectors v1-0:JST-XH-04-PACKAGE-LONG-PAD
- added U$4: TERMINAL_4P, TA_library:TERMINAL_4P
- C1: value (none) -> 22u
- C2: value (none) -> 100n
- C3: value (none) -> 4.7uF
- D4: value (none) -> LED_G
- NPN: value (none) -> BS170
- moved U$3 99.5 mm to (5.99, 59.7), turned to 270 degrees
- moved JP8 71.4 mm to (8.41, 118.3)
- moved JP2 55.5 mm to (61.2, 74.8), turned to 0 degrees
- moved JP4 43.2 mm to (70.2, 77.1)
- moved MINI1 41.9 mm to (28.9, 41.7)
- moved JP7 34.7 mm to (74.5, 81.9), turned to 0 degrees
- moved D4 31.0 mm to (50.4, 75.0), turned to 270 degrees
- moved 330 18.3 mm to (34.7, 62.7), turned to 0 degrees
- moved 1K 18.3 mm to (35.6, 45.0), turned to 180 degrees
- moved NPN 17.0 mm to (35.9, 55.0)
- moved D7 16.5 mm to (35.8, 48.8)
- moved K1 14.3 mm to (54.2, 51.3), turned to 270 degrees
- moved C2 8.98 mm to (57.8, 67.1)
- moved C3 7.76 mm to (37.4, 80.7), turned to 0 degrees
- moved C1 6.48 mm to (49.9, 67.1), flipped to the top
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Connections:
- removed net AC: K1.COM
- removed net AC_IN_1: K1.NO
- removed net CUR_SENSE: U$2.A0, X3.3
- removed net N$4: JP2.1
- removed net N$5: JP2.3
- removed net N$6: JP2.5
- removed net RX: U$3.RX
- removed net TEMP: U$2.A2, X2.2
- removed net TEMP1: X1.5
- removed net TX: U$3.TX
- removed net VOL_SENSE: U$2.A1, X3.4
- new net AC+: HI_LINK1.AC+, U$4.P$2, U$4.P$3
- new net AC-: HI_LINK1.AC-, K1.COM, U$4.P$1
- new net AC_OUT_CHG: K1.NO, U$4.P$4
- new net CURRENT_SENSE: CHARGER.6, SENSING.3, U$2.A0
- new net N$2: FAN.1
- new net TEMP_SENSE: CHARGER.5, TEMP.2, U$2.A2
- new net VOLTAGE_SENSE: CHARGER.7, SENSING.4, U$2.A1
- net 12V: now also CHARGER.1, FAN.3; no longer X1.1, X8.3
- net 5V: now also 5V.1, 5V.2, 5V.3, 5V.4, 5V.5, C5.+, CHARGER.2, SENSING.1, TEMP.1; no longer X1.2, X2.1, X3.1
- net BLU_KANAN: now also LED_R.3; no longer X6.2
- net BLU_KIRI: now also LED_L.3; no longer X5.2
- net DETEKSI_BATERAI_KANAN: now also DB_R.1; no longer X12.1
- net DETEKSI_BATERAI_KIRI: now also DB_L.1; no longer X11.1
- net GND: now also C5.-, CHARGER.8, CHGMODE.2, DB_L.2, DB_R.2, FAN.2, GND.1, GND.2, GND.3, GND.4, GND.5, JP2.5, LED_L.4, LED_R.4, SENSING.2, TEMP.3; no longer JP3.1, U$1.38, X1.6, X10.2, X11.2, X12.2, X2.3, X3.2, X5.1, X6.1, X8.2
- net GRN_KANAN: now also LED_R.1; no longer X6.4
- net GRN_KIRI: now also LED_L.1; no longer X5.4
- net PWM_DISCHARGE: now also CHARGER.4; no longer X1.4
- net PWM_MOSFET: now also CHARGER.3; no longer X1.3
- net RED_KANAN: now also LED_R.2; no longer X6.3
- net RED_KIRI: now also LED_L.2; no longer X5.3
- net RX_BMS: now also JP2.1
- net RX_IOT: now also U$3.RX
- net SWITCH_MODE_DAYA: now also CHGMODE.1; no longer X10.1
- net TX_BMS: now also JP2.3
- net TX_IOT: now also U$3.TX
Routing:
- net GND: track 0.00 -> 411.2 mm
- net 12V: track 0.00 -> 315.3 mm, vias 0 -> 5
- net 5V: track 0.00 -> 264.2 mm, vias 0 -> 2
- net CURRENT_SENSE: track 0.00 -> 210.0 mm, vias 0 -> 4
- net TX_BMS: track 0.00 -> 205.0 mm
- net PWM_DISCHARGE: track 0.00 -> 200.1 mm, vias 0 -> 1
- net VOLTAGE_SENSE: track 0.00 -> 148.6 mm, vias 0 -> 8
- net TEMP_SENSE: track 0.00 -> 143.1 mm, vias 0 -> 4
- net GRN_KANAN: track 0.00 -> 142.4 mm, vias 0 -> 1
- net GRN_KIRI: track 0.00 -> 129.0 mm, vias 0 -> 4
- net PWM_MOSFET: track 0.00 -> 127.5 mm, vias 0 -> 1
- net BLU_KANAN: track 0.00 -> 118.1 mm
- net RED_KANAN: track 0.00 -> 110.2 mm, vias 0 -> 4
- net DETEKSI_BATERAI_KIRI: track 0.00 -> 87.7 mm, vias 0 -> 3
- net RED_KIRI: track 0.00 -> 85.7 mm
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- added copper zone on layer 1, net GND
- added copper zone on layer 16, net GND
Other:
- board size 86.4 x 136.6 mm -> 84.3 x 132.8 mm
- board text added: "A3_ADC"
- board text added: "AC+"
- board text added: "AC-"
- board text added: "CHG+"
- board text added: "CHG-"

Commit message: Buat board charger V4
Parts:
- moved GND 0.12 mm to (67.3, 62.3)
- moved CHARGER 0.12 mm to (77.5, 67.4)
- moved DB_R 0.12 mm to (62.3, 127.1)
- moved FAN 0.12 mm to (72.4, 127.1)
- moved LED_L 0.12 mm to (77.5, 48.4)
- moved LED_R 0.12 mm to (68.6, 48.4)
- moved SENSING 0.12 mm to (41.9, 127.1)
- moved 5V 0.12 mm to (25.4, 81.4)
- moved MINI1 0.12 mm to (28.9, 41.8)
- moved U$4 0.12 mm to (67.3, 11.5)
- moved U$3 0.12 mm to (6.02, 59.8)
- moved 1K 0.12 mm to (35.6, 45.1)
- moved 330 0.12 mm to (34.7, 62.8)
- moved C1 0.12 mm to (49.9, 67.2)
- moved C2 0.12 mm to (57.9, 67.2)
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